File: pcb/PMG.kicad_sch (KiCad schematic)
At the start: 60 parts, among them J3 Conn_01x02_Pin, Q1 BC547, Q10 BC547, Q2 BC547, Q3 BC547, Q4 BC547, Q5 BC547, Q6 BC547, Q7 BC547, Q8 BC547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

Commit message: Update to KiCAD 9
Other:
- moved on the sheet: FID1, FID2, FID3, FID4

Commit message: Rename/Remove bom fields
Parts:
- C1: HTL (none) -> 100358; Vendor HTL -> (none); VendorId 100358 -> (none)
- C2, C3, C4, C5: HTL (none) -> 100345; Vendor HTL -> (none); VendorId 100345 -> (none)
- C6: HTL (none) -> 103390; Vendor HTL -> (none); VendorId 103390 -> (none)
- D1, D10, D11, D12, D13, D14, D15, D2, D3, D4, D5, D6, D7, D8, D9: HTL (none) -> 100176; Vendor HTL -> (none); VendorId 100176 -> (none)
- FID1, FID2, FID3, FID4: now left out of the parts list
- J3: HTL (none) -> 101521; Vendor HTL -> (none); VendorId 101521 -> (none)
- MK1: HTL (none) -> 100477; Vendor HTL -> (none); VendorId 100477 -> (none)
- Q1, Q10, Q2, Q3, Q4, Q5, Q6, Q7, Q8, Q9: HTL (none) -> 100215; Vendor HTL -> (none); VendorId 100215 -> (none)
- R1, R2, R23, R3, R4, R5, R6, R7: HTL (none) -> 102798; Vendor HTL -> (none); VendorId 102798 -> (none)
- R10, R11, R12, R13, R14, R15, R16, R20, R8, R9: HTL (none) -> 102812; Vendor HTL -> (none); VendorId 102812 -> (none)
- R17, R21: HTL (none) -> 102836; Vendor HTL -> (none); VendorId 102836 -> (none)
- R18: HTL (none) -> 102819; Vendor HTL -> (none); VendorId 102819 -> (none)
- R19: HTL (none) -> 102845; Vendor HTL -> (none); VendorId 102845 -> (none)
- R22: HTL (none) -> 102795; Vendor HTL -> (none); VendorId 102795 -> (none)
